Commit message: Adjusted propulsion plugin to work with current controller and updated component_snippets for ADIS IMU

File: rotors_description/urdf/component_snippets.xacro (robot description, xacro)
@@ -18,14 +18,4 @@
 <robot xmlns:xacro="http://ros.org/wiki/xacro">
   <xacro:property name="pi" value="3.14159265359" />
-  <!-- Macro for the inertia of a box -->
-  <xacro:macro name="box_inertia" params="x y z mass">
-    <inertia ixx="${0.0833333 * mass * (y*y + z*z)}" ixy="0.0" ixz="0.0"
-      iyy="${0.0833333 * mass * (x*x + z*z)}" iyz="0.0"
-      izz="${0.0833333 * mass * (x*x + y*y)}" />
-  </xacro:macro>
-  <!-- Macro for the inertia of a cube -->
-  <xacro:macro name="cube_inertia" params="l mass">
-    <xacro:box_inertia x="${l}" y="${l}" z="${l}" mass="${mass}" />
-  </xacro:macro>
   <!-- Macro to add logging to a bag file. -->
   <xacro:macro name="bag_plugin_macro"
@@ -49,5 +39,5 @@
     <link name="${namespace}/camera_${camera_suffix}_link">
       <collision>
-        <origin xyz="0 0 0" rpy="0 ${pi/2} 0" />
+        <origin xyz="0 0 0" rpy="0 0 0" />
         <geometry>
           <xacro:insert_block name="geometry" />
@@ -121,80 +111,4 @@
     </gazebo>
   </xacro:macro>
-  <!-- Macro to add a camera. 2 (configurable mass, no massless links) -->
-  <xacro:macro name="camera_macro_2"
-    params="namespace parent_link camera_suffix frame_rate
-      horizontal_fov image_width image_height image_format min_distance
-      max_distance noise_mean noise_stddev mass enable_visual *geometry *inertia *origin">
-    <link name="${namespace}/camera_${camera_suffix}_link">
-    <xacro:if value="${enable_visual}">
-      <visual>
-        <origin xyz="0 0 0" rpy="0 ${pi/2} 0" />
-        <geometry>
-          <xacro:insert_block name="geometry" />
-        </geometry>
-        <material name="red" />
-      </visual>
-    </xacro:if>
-      <inertial>
-        <mass value="${mass-0.001}" />
-        <origin xyz="0 0 0" rpy="0 0 0" />
-        <xacro:insert_block name="inertia" />
-      </inertial>
-    </link>
-    <joint name="${namespace}/camera_${camera_suffix}_joint" type="fixed">
-      <xacro:insert_block name="origin" />
-      <parent link="${parent_link}" />
-      <child link="${namespace}/camera_${camera_suffix}_link" />
-    </joint>
-    <link name="${namespace}/camera_${camera_suffix}_optical_link">
-    <inertial>
-      <mass value="0.001" />
-      <origin xyz="0 0 0" rpy="0 0 0" />
-      <xacro:cube_inertia l="0.02" mass="0.001" />
-    </inertial>
-    </link>
-    <joint name="${namespace}/camera_${camera_suffix}_optical_joint" type="fixed" >
-      <origin xyz="0 0 0" rpy="${-pi/2} 0 ${-pi/2}" />
-      <parent link="${namespace}/camera_${camera_suffix}_link" />
-      <child link="${namespace}/camera_${camera_suffix}_optical_link" />
-    </joint>
-    <gazebo reference="${namespace}/camera_${camera_suffix}_link">
-      <sensor type="camera" name="${namespace}_camera_${camera_suffix}">
-        <update_rate>${frame_rate}</update_rate>
-        <camera name="head">
-          <horizontal_fov>${horizontal_fov}</horizontal_fov>
-          <image>
-            <width>${image_width}</width>
-            <height>${image_height}</height>
-            <format>${image_format}</format>
-          </image>
-          <clip>
-            <near>${min_distance}</near>
-            <far>${max_distance}</far>
-          </clip>
-          <noise>
-            <type>gaussian</type>
-            <mean>${noise_mean}</mean>
-            <stddev>${noise_stddev}</stddev>
-          </noise>
-        </camera>
-        <plugin name="${namespace}_camera_${camera_suffix}_controller" filename="libgazebo_ros_camera.so">
-          <robotNamespace>${namespace}</robotNamespace>
-          <alwaysOn>true</alwaysOn>
-          <updateRate>${frame_rate}</updateRate>
-          <cameraName>cam_${camera_suffix}</cameraName>
-          <imageTopicName>image_raw</imageTopicName>
-          <cameraInfoTopicName>camera_info</cameraInfoTopicName>
-          <frameName>camera_${camera_suffix}_link</frameName>
-          <hackBaseline>0.7</hackBaseline>
-          <distortionK1>0.0</distortionK1>
-          <distortionK2>0.0</distortionK2>
-          <distortionK3>0.0</distortionK3>
-          <distortionT1>0.0</distortionT1>
-          <distortionT2>0.0</distortionT2>
-        </plugin>
-      </sensor>
-    </gazebo>
-  </xacro:macro>
   <!-- Camera joint macro - just the joints, links, and collisions for a single
        camera. -->
@@ -335,6 +249,5 @@
   <!-- ==================== ROS INTERFACE MACRO ====================== -->
   <!-- =============================================================== -->
-  <!--
-  <xacro:macro
+  <!-- <xacro:macro
   		name="ros_interface_plugin_macro"
   		params="namespace">
@@ -344,6 +257,5 @@
       </plugin>
     </gazebo>
-  </xacro:macro>
-  -->
+  </xacro:macro>-->
   <!-- =============================================================== -->
   <!-- ================== MAVLINK INTERFACE MACRO ==================== -->
@@ -417,51 +329,4 @@
     </gazebo>
   </xacro:macro>
-  <!-- Macro to add an IMU (using Gazebo IMU) -->
-  <xacro:macro name="imu_s_plugin_macro"
-  params="namespace imu_suffix parent_link imu_topic
-    mass_imu_sensor *inertia *origin">
-  <!-- IMU link -->
-  <link name="${namespace}/imu${imu_suffix}_link">
-    <inertial>
-      <xacro:insert_block name="inertia" />
-      <mass value="${mass_imu_sensor}" />  <!-- [kg] -->
-      <origin xyz="0 0 0" rpy="0 0 0" />
-    </inertial>
-  </link>
-  <!-- IMU joint -->
-  <joint name="${namespace}/imu${imu_suffix}_joint" type="revolute">
-    <xacro:insert_block name="origin" />
-    <parent link="${parent_link}" />
-    <child link="${namespace}/imu${imu_suffix}_link" />
-    <limit upper="0" lower="0" effort="0" velocity="0" />
-  </joint>
-  <gazebo reference="${namespace}/imu${imu_suffix}_link">
-    <gravity>true</gravity>
-    <sensor name="imu_sensor" type="imu">
-      <pose>0 0 0 0 0 0</pose>
-      <always_on>true</always_on>
-      <visualize>true</visualize>
-      <topic>__default_topic__</topic>
-      <update_rate>100</update_rate>
-      <imu>
-        <angular_velocity>
-          <x></x>
-          <y></y>
-          <y></y>
-        </angular_velocity>
-        <linear_acceleration>
-          <x></x>
-          <y></y>
-          <y></y>
-        </linear_acceleration>
-      </imu>
-      <plugin filename="librotors_gazebo_imu_s_plugin.so" name="rotors_gazebo_imu_s_plugin">
-        <robotNamespace>${namespace}</robotNamespace> <!-- (string, required): ros namespace in which the messages are published -->
-        <linkName>${namespace}/imu${imu_suffix}_link</linkName> <!-- (string, required): name of the body which holds the IMU sensor -->
-        <imuTopic>${imu_topic}</imuTopic> <!-- (string): name of the sensor output topic and prefix of service names (defaults to imu) -->
-      </plugin>
-    </sensor>
-  </gazebo>
-  </xacro:macro>
   <!-- Macro to add a generic odometry sensor. -->
   <xacro:macro name="odometry_plugin_macro"
@@ -522,5 +387,5 @@
     params="namespace gps_suffix parent_link gps_topic ground_speed_topic
       mass_gps_sensor horizontal_pos_std_dev vertical_pos_std_dev
-      horizontal_vel_std_dev vertical_vel_std_dev enable_delay *inertia *origin">
+      horizontal_vel_std_dev vertical_vel_std_dev *inertia *origin">
     <!-- GPS link -->
     <link name="${namespace}/gps${gps_suffix}_link">
@@ -543,4 +408,5 @@
         <visualize>0</visualize>
         <always_on>1</always_on>
+        <update_rate>5</update_rate>
         <gps>
           <position_sensing>
@@ -590,66 +456,4 @@
           <horVelStdDev>${horizontal_vel_std_dev}</horVelStdDev> <!-- standard deviation for horizontal speed noise [m/s] -->
           <verVelStdDev>${vertical_vel_std_dev}</verVelStdDev> <!-- standard deviation for vertical speed noise [m/s] -->
-          <enableDelay>${enable_delay}</enableDelay>
-          <updateInterval>0.10</updateInterval>
-          <delay>0.12</delay>
-          <!--<rqstFwdToRos>${rqst_fwd_to_ros}</rqstFwdToRos>-->
-        </plugin>
-      </sensor>
-    </gazebo>
-  </xacro:macro>
-  <!-- Macro to add a single-ray LIDAR. -->
-  <xacro:macro name="lidar_plugin_macro"
-    params="namespace lidar_suffix mass_lidar_sensor
-            parent_link lidar_topic n_hrz n_vrt
-            rng_min rng_max ang_min_hrz ang_max_hrz
-            ang_min_vrt ang_max_vrt noise_std *inertia *origin">
-    <!-- LIDAR link -->
-    <link name="${namespace}/lidar${lidar_suffix}_link">
-      <inertial>
-        <xacro:insert_block name="inertia" />
-        <mass value="${mass_lidar_sensor}" />  <!-- [kg] -->
-        <origin xyz="0 0 0" rpy="0 0 0" />
-      </inertial>
-    </link>
-    <!-- LIDAR joint -->
-    <joint name="${namespace}/lidar${lidar_suffix}_joint" type="revolute">
-      <xacro:insert_block name="origin" />
-      <parent link="${parent_link}" />
-      <child link="${namespace}/lidar${lidar_suffix}_link" />
-      <limit upper="0" lower="0" effort="0" velocity="0" />
-    </joint>
-    <gazebo reference="${namespace}/lidar${lidar_suffix}_link">
-      <sensor type="ray" name="${namespace}_lidar${lidar_suffix}">
-        <pose>0 0 0 0 0 0</pose>
-        <visualize>1</visualize>
-        <always_on>1</always_on>
-        <ray>
-          <scan>
-            <horizontal>
-              <samples>${n_hrz}</samples>
-              <resolution>1</resolution>
-              <min_angle>${ang_min_hrz}</min_angle>
-              <max_angle>${ang_max_hrz}</max_angle>
-            </horizontal>
-            <vertical>
-              <samples>${n_vrt}</samples>
-              <resolution>1</resolution>
-              <min_angle>${ang_min_vrt}</min_angle>
-              <max_angle>${ang_max_vrt}</max_angle>
-            </vertical>
-          </scan>
-          <range>
-            <min>${rng_min}</min>
-            <max>${rng_max}</max>
-          </range>
-          <noise>
-            <type>gaussian</type>
-            <mean>0</mean>
-            <stddev>${noise_std}</stddev>
-          </noise>
-        </ray>
-        <plugin filename="librotors_gazebo_lidar_plugin.so" name="rotors_gazebo_lidar${lidar_suffix}_plugin">
-          <robotNamespace>${namespace}</robotNamespace>
-          <lidarTopic>${lidar_topic}</lidarTopic>
         </plugin>
       </sensor>
@@ -957,73 +761,4 @@
     </xacro:imu_plugin_macro>
   </xacro:macro>
-  <!-- Techpod Mono-VI Sensor Macro -->
-  <xacro:macro name="asl_mono_vi_1" params="namespace parent_link suffix fps h_fov imu_topic acc_nd acc_rw gyr_nd gyr_rw *T_base_cam *T_cam_imu *T_cam_odom">
-    <xacro:camera_macro_2
-      namespace="${namespace}"
-      parent_link="${parent_link}"
-      camera_suffix="${suffix}"
-      frame_rate="${fps}"
-      horizontal_fov="${h_fov}"
-      image_width="752"
-      image_height="480"
-      image_format="L8"
-      min_distance="0.02"
-      max_distance="8000"
-      noise_mean="0.0"
-      noise_stddev="0.007"
-      mass="0.02"
-      enable_visual="true">
-      <mesh filename="package://rotors_description/meshes/vi_camera.dae" scale="1 1 1" />
-      <xacro:cube_inertia l="0.02" mass="0.01" />
-      <xacro:insert_block name="T_base_cam" />
-    </xacro:camera_macro_2>
-    <xacro:imu_plugin_macro
-      namespace="${namespace}"
-      imu_suffix="_camera_${suffix}"
-      parent_link="${namespace}/camera_${suffix}_optical_link"
-      imu_topic="${imu_topic}"
-      mass_imu_sensor="0.01"
-      gyroscope_noise_density="${gyr_nd}"
-      gyroscope_random_walk="${gyr_rw}"
-      gyroscope_bias_correlation_time="1000.0"
-      gyroscope_turn_on_bias_sigma="0.0087"
-      accelerometer_noise_density="${acc_nd}"
-      accelerometer_random_walk="${acc_rw}"
-      accelerometer_bias_correlation_time="300.0"
-      accelerometer_turn_on_bias_sigma="0.1960">
-      <xacro:cube_inertia l="0.02" mass="0.01" />
-      <xacro:insert_block name="T_cam_imu"/>
-    </xacro:imu_plugin_macro>
-    <xacro:odometry_plugin_macro
-      namespace="${namespace}"
-      odometry_sensor_suffix="_camera_${suffix}"
-      parent_link="${namespace}/camera_${suffix}_optical_link"
-      pose_topic="cam_${suffix}/pose"
-      pose_with_covariance_topic="cam_${suffix}/t1"
-      position_topic="cam_${suffix}/t2"
-      transform_topic="cam_${suffix}/t3"
-      odometry_topic="cam_${suffix}/odometry"
-      parent_frame_id="world"
-      child_frame_id="odometry_sensor_camera_${suffix}"
-      mass_odometry_sensor="0.001"
-      measurement_divisor="1"
-      measurement_delay="0"
-      unknown_delay="0.0"
-      noise_normal_position="0 0 0"
-      noise_normal_quaternion="0 0 0"
-      noise_normal_linear_velocity="0 0 0"
-      noise_normal_angular_velocity="0 0 0"
-      noise_uniform_position="0 0 0"
-      noise_uniform_quaternion="0 0 0"
-      noise_uniform_linear_velocity="0 0 0"
-      noise_uniform_angular_velocity="0 0 0"
-      enable_odometry_map="false"
-      odometry_map=""
-      image_scale="">
-      <xacro:cube_inertia l="0.02" mass="0.001" />
-      <xacro:insert_block name="T_cam_odom"/>
-    </xacro:odometry_plugin_macro>
-    <!---->
-  </xacro:macro>
   <xacro:macro name="ground_truth_imu_and_odometry" params="namespace parent_link">
     <!-- Mount an IMU providing ground truth. -->
@@ -1072,9 +807,9 @@
       odometry_map=""
       image_scale="">
-      <xacro:cube_inertia l="0.001" mass="0.00001" /> <!-- [kg m^2] [kg m^2] [kg m^2] [kg m^2] [kg m^2] [kg m^2] -->
+      <inertia ixx="0.00001" ixy="0.0" ixz="0.0" iyy="0.00001" iyz="0.0" izz="0.00001" /> <!-- [kg m^2] [kg m^2] [kg m^2] [kg m^2] [kg m^2] [kg m^2] -->
       <origin xyz="0.0 0.0 0.0" rpy="0.0 0.0 0.0" />
     </xacro:odometry_plugin_macro>
   </xacro:macro>
-  <xacro:macro name="default_imu" params="namespace parent_link *origin">
+  <xacro:macro name="default_imu" params="namespace parent_link">
     <!-- ADIS16448 IMU. -->
     <xacro:imu_plugin_macro
@@ -1092,50 +827,10 @@
       accelerometer_bias_correlation_time="300.0"
       accelerometer_turn_on_bias_sigma="0.1960">
-      <xacro:cube_inertia l="0.02" mass="0.015" />
-      <xacro:insert_block name="origin" />
+      <inertia ixx="0.00001" ixy="0.0" ixz="0.0" iyy="0.00001" iyz="0.0" izz="0.00001" />
+      <origin xyz="0 0 0" rpy="0 0 0" />
     </xacro:imu_plugin_macro>
   </xacro:macro>
-  <xacro:macro name="ideal_imu" params="namespace parent_link *origin">
-    <xacro:imu_plugin_macro
-      namespace="${namespace}"
-      imu_suffix=""
-      parent_link="${parent_link}"
-      imu_topic="imu"
-      mass_imu_sensor="0.015"
-      gyroscope_noise_density="0.0"
-      gyroscope_random_walk="0.0"
-      gyroscope_bias_correlation_time="10000.0"
-      gyroscope_turn_on_bias_sigma="0.0"
-      accelerometer_noise_density="0.0"
-      accelerometer_random_walk="0.0"
-      accelerometer_bias_correlation_time="10000.0"
-      accelerometer_turn_on_bias_sigma="0.0">
-      <xacro:cube_inertia l="0.02" mass="0.015" />
-      <xacro:insert_block name="origin" />
-    </xacro:imu_plugin_macro>
-  </xacro:macro>
-  <xacro:macro name="default_camera" params="namespace parent_link camera_suffix *origin">
-    <xacro:camera_macro_2
-      namespace="${namespace}"
-      parent_link="${parent_link}"
-      camera_suffix="${camera_suffix}"
-      frame_rate="30"
-      horizontal_fov="1.3962634"
-      image_width="752"
-      image_height="480"
-      image_format="L8"
-      min_distance="0.02"
-      max_distance="8000"
-      noise_mean="0.0"
-      noise_stddev="0.007"
-      mass = "0.01"
-      enable_visual="true">
-      <mesh filename="package://rotors_description/meshes/vi_camera.dae" scale="1 1 1" />
-      <xacro:cube_inertia l="0.02" mass="0.01" />
-      <xacro:insert_block name="origin" />
-    </xacro:camera_macro_2>
-  </xacro:macro>
-  <xacro:macro name="default_gps" params="namespace parent_link *origin">
-    <!-- Default GPS including ground truth GPS -->
+  <xacro:macro name="default_gps" params="namespace parent_link">
+    <!-- Default GPS. -->
     <xacro:gps_plugin_macro
       namespace="${namespace}"
@@ -1148,55 +843,8 @@
       vertical_pos_std_dev="6.0"
       horizontal_vel_std_dev="0.1"
-      vertical_vel_std_dev="0.1"
-      enable_delay = "true">
-      <xacro:cube_inertia l="0.02" mass="0.015" />
-      <xacro:insert_block name="origin" />
+      vertical_vel_std_dev="0.1">
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
File: rotors_description/urdf/multirotor_base_advanced.xacro (robot description, xacro)
@@ -75,5 +75,5 @@
   <!-- Rotor joint and link -->
   <xacro:macro name="vertical_rotor_advanced"
-    params="robot_namespace suffix direction parent mass_rotor radius_rotor time_constant_up time_constant_down max_rot_velocity dead_rot_velocity motor_number color use_own_mesh mesh *origin *inertia">
+    params="robot_namespace suffix direction x y z parent mass_rotor radius_rotor time_constant_up time_constant_down max_rot_velocity dead_rot_velocity motor_number color use_own_mesh mesh *origin *inertia">
     <joint name="${robot_namespace}/rotor_${motor_number}_joint" type="continuous">
       <xacro:insert_block name="origin" />
@@ -130,5 +130,5 @@
           <jointName>${robot_namespace}/rotor_${motor_number}_joint</jointName>
           <linkNameParent>${namespace}/base_link</linkNameParent>
-          <cp>0 0 4</cp>
+          <cp>${x} ${y} ${z}</cp>
           <axisPosRot>0 0 -1</axisPosRot>
           <turnDir>${direction}</turnDir>

File: rotors_description/urdf/peregrine.xacro (robot description, xacro)
@@ -41,7 +41,4 @@
   <xacro:property name="rotor_drag_coefficient" value="12.06428e-05" />
   <xacro:property name="rolling_moment_coefficient" value="0.000001" />
-  <!-- <xacro:property name="length_rod" value="1.45" /> [m] -->
-  <!-- <xacro:property name="diameter_rod" value="0.004" /> [m] -->
-  <!-- <xacro:property name="diameter_ball" value="0.11" />  [m] -->
   <!-- Property Blocks -->
   <xacro:property name="body_inertia">
@@ -70,5 +67,5 @@
     suffix="front_left"
     direction="ccw"
-    x = ${cos30*arm_length} y = ${sin30*arm_length} z = ${rotor_offset_top}
+    x = "${cos30*arm_length}" y = "${sin30*arm_length}" z = "${rotor_offset_top}"
     parent="${namespace}/base_link"
     mass_rotor="${mass_rotor}"
@@ -89,5 +86,5 @@
     suffix="left"
     direction="cw"
-    x = 0 y = ${arm_length} z = ${rotor_offset_top}
+    x = "0" y = "${arm_length}" z = "${rotor_offset_top}"
     parent="${namespace}/base_link"
     mass_rotor="${mass_rotor}"
@@ -108,5 +105,5 @@
     suffix="back_left"
     direction="ccw"
-    x = -${cos30*arm_length} y = ${sin30*arm_length} z = ${rotor_offset_top}
+    x = "-${cos30*arm_length}" y = "${sin30*arm_length}" z = "${rotor_offset_top}"
     parent="${namespace}/base_link"
     mass_rotor="${mass_rotor}"
@@ -127,5 +124,5 @@
     suffix="back_right"
     direction="cw"
-    x = -${cos30*arm_length} y = -${sin30*arm_length} z = ${rotor_offset_top}
+    x = "-${cos30*arm_length}" y = "-${sin30*arm_length}" z = "${rotor_offset_top}"
     parent="${namespace}/base_link"
     mass_rotor="${mass_rotor}"
@@ -146,5 +143,5 @@
     suffix="right"
     direction="ccw"
-    x=0 y=-${arm_length} z=${rotor_offset_top}
+    x="0" y="-${arm_length}" z="${rotor_offset_top}"
     parent="${namespace}/base_link"
     mass_rotor="${mass_rotor}"
@@ -165,5 +162,5 @@
     suffix="front_right"
     direction="cw"
-    x = ${cos30*arm_length} y = -${sin30*arm_length} z = ${rotor_offset_top}
+    x = "${cos30*arm_length}" y = "-${sin30*arm_length}" z = "${rotor_offset_top}"
     parent="${namespace}/base_link"
     mass_rotor="${mass_rotor}"

File: rotors_description/urdf/peregrine_base.xacro (robot description, xacro)
@@ -28,5 +28,4 @@
     <xacro:default_mavlink_interface namespace="${namespace}" imu_sub_topic="imu" rotor_count="6" />
   </xacro:if>
-  <!-- Mount an ADIS16448 IMU. -->
   <xacro:default_imu namespace="${namespace}" parent_link="${namespace}/base_link" />
   <xacro:if value="$(arg enable_ground_truth)">
