Commit message: Propulsion Plugin Working, Not Building Mavlink (CMAKE edited)

File: rotors_description/urdf/component_snippets.xacro (robot description, xacro)
@@ -18,4 +18,14 @@
 <robot xmlns:xacro="http://ros.org/wiki/xacro">
   <xacro:property name="pi" value="3.14159265359" />
+  <!-- Macro for the inertia of a box -->
+  <xacro:macro name="box_inertia" params="x y z mass">
+    <inertia ixx="${0.0833333 * mass * (y*y + z*z)}" ixy="0.0" ixz="0.0"
+      iyy="${0.0833333 * mass * (x*x + z*z)}" iyz="0.0"
+      izz="${0.0833333 * mass * (x*x + y*y)}" />
+  </xacro:macro>
+  <!-- Macro for the inertia of a cube -->
+  <xacro:macro name="cube_inertia" params="l mass">
+    <xacro:box_inertia x="${l}" y="${l}" z="${l}" mass="${mass}" />
+  </xacro:macro>
   <!-- Macro to add logging to a bag file. -->
   <xacro:macro name="bag_plugin_macro"
@@ -102,4 +112,80 @@
           <frameName>camera_${camera_suffix}_link</frameName>
           <hackBaseline>0.0</hackBaseline>
+          <distortionK1>0.0</distortionK1>
+          <distortionK2>0.0</distortionK2>
+          <distortionK3>0.0</distortionK3>
+          <distortionT1>0.0</distortionT1>
+          <distortionT2>0.0</distortionT2>
+        </plugin>
+      </sensor>
+    </gazebo>
+  </xacro:macro>
+  <!-- Macro to add a camera. 2 (configurable mass, no massless links) -->
+  <xacro:macro name="camera_macro_2"
+    params="namespace parent_link camera_suffix frame_rate
+      horizontal_fov image_width image_height image_format min_distance
+      max_distance noise_mean noise_stddev mass enable_visual *geometry *inertia *origin">
+    <link name="${namespace}/camera_${camera_suffix}_link">
+    <xacro:if value="${enable_visual}">
+      <visual>
+        <origin xyz="0 0 0" rpy="0 ${pi/2} 0" />
+        <geometry>
+          <xacro:insert_block name="geometry" />
+        </geometry>
+        <material name="red" />
+      </visual>
+    </xacro:if>
+      <inertial>
+        <mass value="${mass-0.001}" />
+        <origin xyz="0 0 0" rpy="0 0 0" />
+        <xacro:insert_block name="inertia" />
+      </inertial>
+    </link>
+    <joint name="${namespace}/camera_${camera_suffix}_joint" type="fixed">
+      <xacro:insert_block name="origin" />
+      <parent link="${parent_link}" />
+      <child link="${namespace}/camera_${camera_suffix}_link" />
+    </joint>
+    <link name="${namespace}/camera_${camera_suffix}_optical_link">
+    <inertial>
+      <mass value="0.001" />
+      <origin xyz="0 0 0" rpy="0 0 0" />
+      <xacro:cube_inertia l="0.02" mass="0.001" />
+    </inertial>
+    </link>
+    <joint name="${namespace}/camera_${camera_suffix}_optical_joint" type="fixed" >
+      <origin xyz="0 0 0" rpy="${-pi/2} 0 ${-pi/2}" />
+      <parent link="${namespace}/camera_${camera_suffix}_link" />
+      <child link="${namespace}/camera_${camera_suffix}_optical_link" />
+    </joint>
+    <gazebo reference="${namespace}/camera_${camera_suffix}_link">
+      <sensor type="camera" name="${namespace}_camera_${camera_suffix}">
+        <update_rate>${frame_rate}</update_rate>
+        <camera name="head">
+          <horizontal_fov>${horizontal_fov}</horizontal_fov>
+          <image>
+            <width>${image_width}</width>
+            <height>${image_height}</height>
+            <format>${image_format}</format>
+          </image>
+          <clip>
+            <near>${min_distance}</near>
+            <far>${max_distance}</far>
+          </clip>
+          <noise>
+            <type>gaussian</type>
+            <mean>${noise_mean}</mean>
+            <stddev>${noise_stddev}</stddev>
+          </noise>
+        </camera>
+        <plugin name="${namespace}_camera_${camera_suffix}_controller" filename="libgazebo_ros_camera.so">
+          <robotNamespace>${namespace}</robotNamespace>
+          <alwaysOn>true</alwaysOn>
+          <updateRate>${frame_rate}</updateRate>
+          <cameraName>cam_${camera_suffix}</cameraName>
+          <imageTopicName>image_raw</imageTopicName>
+          <cameraInfoTopicName>camera_info</cameraInfoTopicName>
+          <frameName>camera_${camera_suffix}_link</frameName>
+          <hackBaseline>0.7</hackBaseline>
           <distortionK1>0.0</distortionK1>
           <distortionK2>0.0</distortionK2>
@@ -831,4 +917,25 @@
     </xacro:imu_plugin_macro>
   </xacro:macro>
+  <xacro:macro name="default_camera" params="namespace parent_link camera_suffix *origin">
+   <xacro:camera_macro_2
+     namespace="${namespace}"
+     parent_link="${parent_link}"
+     camera_suffix="${camera_suffix}"
+     frame_rate="30"
+     horizontal_fov="1.3962634"
+     image_width="752"
+     image_height="480"
+     image_format="L8"
+     min_distance="0.02"
+     max_distance="8000"
+     noise_mean="0.0"
+     noise_stddev="0.007"
+     mass = "0.01"
+     enable_visual="true">
+     <mesh filename="package://rotors_description/meshes/vi_camera.dae" scale="1 1 1" />
+     <xacro:cube_inertia l="0.02" mass="0.01" />
+     <xacro:insert_block name="origin" />
+   </xacro:camera_macro_2>
+ </xacro:macro>
   <xacro:macro name="default_gps" params="namespace parent_link">
     <!-- Default GPS. -->

File: rotors_description/urdf/multirotor_base_advanced.xacro (robot description, xacro)
@@ -69,5 +69,5 @@
         <robotNamespace>${robot_namespace}</robotNamespace>
         <linkName>${robot_namespace}/base_link</linkName>
-        <rotorVelocitySlowdownSim>${rotor_velocity_slowdown_sim}</rotorVelocitySlowdownSim>
+        <!--<rotorVelocitySlowdownSim>${rotor_velocity_slowdown_sim}</rotorVelocitySlowdownSim>-->
       </plugin>
     </gazebo>
@@ -75,5 +75,5 @@
   <!-- Rotor joint and link -->
   <xacro:macro name="vertical_rotor_advanced"
-    params="robot_namespace suffix direction x y z parent mass_rotor radius_rotor time_constant_up time_constant_down max_rot_velocity dead_rot_velocity motor_number color use_own_mesh mesh *origin *inertia">
+    params="robot_namespace direction parent mass_rotor radius_rotor motor_number color use_own_mesh mesh *origin *inertia">
     <joint name="${robot_namespace}/rotor_${motor_number}_joint" type="continuous">
       <xacro:insert_block name="origin" />
@@ -107,9 +107,9 @@
       </collision>
     </link>
-    <gazebo>
-      <!-- changed from original multirotor_base to implement advanced propulsion_plugin -->
+      <!-- <gazebo>
+      changed from original multirotor_base to implement advanced propulsion_plugin
       <plugin name="${robot_namespace}_${suffix}_propulsion" filename="librotors_gazebo_propulsion_plugin.so">
         <robotNamespace>${robot_namespace}</robotNamespace>
-        <!-- changed from original multirotor_base to implement advanced propulsion_plugin
+         changed from original multirotor_base to implement advanced propulsion_plugin
         <jointName>${robot_namespace}/rotor_${motor_number}_joint</jointName>
         <linkName>${robot_namespace}/rotor_${motor_number}</linkName>
@@ -126,5 +126,4 @@
         <motorSpeedPubTopic>motor_speed/${motor_number}</motorSpeedPubTopic>
         <rotorVelocitySlowdownSim>${rotor_velocity_slowdown_sim}</rotorVelocitySlowdownSim>
-        -->
         <prop name="rotor_${motor_number}">
           <jointName>${robot_namespace}/rotor_${motor_number}_joint</jointName>
@@ -136,12 +135,13 @@
           <motorNumber>${motor_number}</motorNumber>
           <propParamsYAML>$(find rotors_gazebo)/resource/peregrine_propconfig.yaml</propParamsYAML>
-          <tauUp>${time_constant_up}</tauUp>       <!-- first-order system timeconstant rev up [s] -->
-          <tauDown>${time_constant_down}</tauDown>   <!-- first-order system timeconstant rev down [s] -->
-          <tauSpoolUp>${time_constant_up}</tauSpoolUp>        <!-- first-order system timeconstant in dead-zone, i.e between speeds 0 and rdpsDead [s]-->
-          <rdpsDead>1</rdpsDead>    <!-- prop speed dead-zone = 0-rdpsDead [rad/s]-->
-          <rdpsMax>${max_rot_velocity}</rdpsMax> <!-- max prop speed [rad/s]-->
+          <tauUp>${time_constant_up}</tauUp>
+          <tauDown>${time_constant_down}</tauDown>
+          <tauSpoolUp>${time_constant_up}</tauSpoolUp>
+          <rdpsDead>1</rdpsDead>
+          <rdpsMax>${max_rot_velocity}</rdpsMax>
         </prop>
       </plugin>
     </gazebo>
+    -->
     <gazebo reference="${robot_namespace}/rotor_${motor_number}">
       <material>Gazebo/${color}</material>
