Commit message: Propulsion Plugin Working, Not Building Mavlink (CMAKE edited)

File: rotors_description/urdf/peregrineC.xacro (robot description, xacro)
@@ -19,5 +19,5 @@
   <!-- Properties -->
   <xacro:property name="namespace" value="$(arg namespace)" />
-  <!-- Slows down rotor vel in simulation s.t. no aliasing -->
+  <!-- What's this? -->
   <xacro:property name="rotor_velocity_slowdown_sim" value="10" />
   <xacro:property name="use_mesh_file" value="true" />
@@ -25,8 +25,9 @@
   <!-- Params to be adjusted from firefly to peregrine -->
   <xacro:property name="mass" value="4.6" /> <!-- [kg] -->
-  <xacro:property name="body_width" value="0.4" /> <!-- [m] -->
-  <xacro:property name="body_height" value="0.4" /> <!-- [m] -->
-  <xacro:property name="mass_rotor" value="0.033" /> <!-- [kg] -->
-  <xacro:property name="arm_length" value="0.42" /> <!-- [m] -->
+  <xacro:property name="body_width" value="0.3" /> <!-- [m] -->
+  <xacro:property name="body_height" value="0.3" /> <!-- [m] -->
+  <xacro:property name="mass_rotor" value="0.008" /> <!-- [kg] -->
+  <xacro:property name="arm_length" value="0.4" /> <!-- [m] -->
+  <!-- this moight cause problems because negative -->
   <xacro:property name="rotor_offset_top" value="-0.05" /> <!-- [m] -->
   <xacro:property name="radius_rotor" value="0.1778" /> <!-- [m] -->
@@ -36,9 +37,11 @@
   <xacro:property name="time_constant_down" value="0.1" /> <!-- [s] -->
   <xacro:property name="max_rot_velocity" value="838" /> <!-- [rad/s] euals 8000rpm -->
-  <xacro:property name="dead_rot_velocity" value="100" />
   <xacro:property name="sin30" value="0.5" />
   <xacro:property name="cos30" value="0.866025403784" />
   <xacro:property name="rotor_drag_coefficient" value="12.06428e-05" />
   <xacro:property name="rolling_moment_coefficient" value="0.000001" />
+  <!-- <xacro:property name="length_rod" value="1.45" /> [m] -->
+  <!-- <xacro:property name="diameter_rod" value="0.004" /> [m] -->
+  <!-- <xacro:property name="diameter_ball" value="0.11" />  [m] -->
   <!-- Property Blocks -->
   <xacro:property name="body_inertia">
@@ -50,5 +53,5 @@
   </xacro:property>
   <!-- Included URDF Files -->
-  <xacro:include filename="$(find rotors_description)/urdf/multirotor_base_advanced.xacro" />
+  <xacro:include filename="$(find rotors_description)/urdf/multirotor_base.xacro" />
   <!-- Instantiate multirotor_base_macro once -->
   <xacro:multirotor_base_macro
@@ -63,9 +66,10 @@
   </xacro:multirotor_base_macro>
   <!-- Instantiate rotors -->
-  <xacro:vertical_rotor_advanced
+  <xacro:vertical_rotor
     robot_namespace="${namespace}"
     suffix="front_left"
     direction="ccw"
-    x = "${cos30*arm_length}" y = "${sin30*arm_length}" z = "${rotor_offset_top}"
+    motor_constant="${motor_constant}"
+    moment_constant="${moment_constant}"
     parent="${namespace}/base_link"
     mass_rotor="${mass_rotor}"
@@ -74,6 +78,7 @@
     time_constant_down="${time_constant_down}"
     max_rot_velocity="${max_rot_velocity}"
-    dead_rot_velocity="${dead_rot_velocity}"
     motor_number="0"
+    rotor_drag_coefficient="${rotor_drag_coefficient}"
+    rolling_moment_coefficient="${rolling_moment_coefficient}"
     color="Red"
     use_own_mesh="false"
@@ -81,10 +86,11 @@
     <origin xyz="${cos30*arm_length} ${sin30*arm_length} ${rotor_offset_top}" rpy="0 0 0" />
     <xacro:insert_block name="rotor_inertia" />
-  </xacro:vertical_rotor_advanced>
-  <xacro:vertical_rotor_advanced
+  </xacro:vertical_rotor>
+  <xacro:vertical_rotor
     robot_namespace="${namespace}"
     suffix="left"
     direction="cw"
-    x = "0" y = "${arm_length}" z = "${rotor_offset_top}"
+    motor_constant="${motor_constant}"
+    moment_constant="${moment_constant}"
     parent="${namespace}/base_link"
     mass_rotor="${mass_rotor}"
@@ -93,6 +99,7 @@
     time_constant_down="${time_constant_down}"
     max_rot_velocity="${max_rot_velocity}"
-    dead_rot_velocity="${dead_rot_velocity}"
     motor_number="1"
+    rotor_drag_coefficient="${rotor_drag_coefficient}"
+    rolling_moment_coefficient="${rolling_moment_coefficient}"
     color="Blue"
     use_own_mesh="false"
@@ -100,10 +107,10 @@
     <origin xyz="0 ${arm_length} ${rotor_offset_top}" rpy="0 0 0" />
     <xacro:insert_block name="rotor_inertia" />
-  </xacro:vertical_rotor_advanced>
-  <xacro:vertical_rotor_advanced
-    robot_namespace="${namespace}"
+  </xacro:vertical_rotor>
+  <xacro:vertical_rotor robot_namespace="${namespace}"
     suffix="back_left"
     direction="ccw"
-    x = "-${cos30*arm_length}" y = "${sin30*arm_length}" z = "${rotor_offset_top}"
+    motor_constant="${motor_constant}"
+    moment_constant="${moment_constant}"
     parent="${namespace}/base_link"
     mass_rotor="${mass_rotor}"
@@ -112,6 +119,7 @@
     time_constant_down="${time_constant_down}"
     max_rot_velocity="${max_rot_velocity}"
-    dead_rot_velocity="${dead_rot_velocity}"
     motor_number="2"
+    rotor_drag_coefficient="${rotor_drag_coefficient}"
+    rolling_moment_coefficient="${rolling_moment_coefficient}"
     color="Blue"
     use_own_mesh="false"
@@ -119,10 +127,10 @@
     <origin xyz="-${cos30*arm_length} ${sin30*arm_length} ${rotor_offset_top}" rpy="0 0 0" />
     <xacro:insert_block name="rotor_inertia" />
-  </xacro:vertical_rotor_advanced>
-  <xacro:vertical_rotor_advanced
-    robot_namespace="${namespace}"
+  </xacro:vertical_rotor>
+  <xacro:vertical_rotor robot_namespace="${namespace}"
     suffix="back_right"
     direction="cw"
-    x = "-${cos30*arm_length}" y = "-${sin30*arm_length}" z = "${rotor_offset_top}"
+    motor_constant="${motor_constant}"
+    moment_constant="${moment_constant}"
     parent="${namespace}/base_link"
     mass_rotor="${mass_rotor}"
@@ -131,6 +139,7 @@
     time_constant_down="${time_constant_down}"
     max_rot_velocity="${max_rot_velocity}"
-    dead_rot_velocity="${dead_rot_velocity}"
     motor_number="3"
+    rotor_drag_coefficient="${rotor_drag_coefficient}"
+    rolling_moment_coefficient="${rolling_moment_coefficient}"
     color="Blue"
     use_own_mesh="false"
@@ -138,10 +147,11 @@
     <origin xyz="-${cos30*arm_length} -${sin30*arm_length} ${rotor_offset_top}" rpy="0 0 0" />
     <xacro:insert_block name="rotor_inertia" />
-  </xacro:vertical_rotor_advanced>
-  <xacro:vertical_rotor_advanced
+  </xacro:vertical_rotor>
+  <xacro:vertical_rotor
     robot_namespace="${namespace}"
     suffix="right"
     direction="ccw"
-    x="0" y="-${arm_length}" z="${rotor_offset_top}"
+    motor_constant="${motor_constant}"
+    moment_constant="${moment_constant}"
     parent="${namespace}/base_link"
     mass_rotor="${mass_rotor}"
@@ -150,6 +160,7 @@
     time_constant_down="${time_constant_down}"
     max_rot_velocity="${max_rot_velocity}"
-    dead_rot_velocity="${dead_rot_velocity}"
     motor_number="4"
+    rotor_drag_coefficient="${rotor_drag_coefficient}"
+    rolling_moment_coefficient="${rolling_moment_coefficient}"
     color="Blue"
     use_own_mesh="false"
@@ -157,10 +168,11 @@
     <origin xyz="0 -${arm_length} ${rotor_offset_top}" rpy="0 0 0" />
     <xacro:insert_block name="rotor_inertia" />
-  </xacro:vertical_rotor_advanced>
-  <xacro:vertical_rotor_advanced
+  </xacro:vertical_rotor>
+  <xacro:vertical_rotor
     robot_namespace="${namespace}"
     suffix="front_right"
     direction="cw"
-    x = "${cos30*arm_length}" y = "-${sin30*arm_length}" z = "${rotor_offset_top}"
+    motor_constant="${motor_constant}"
+    moment_constant="${moment_constant}"
     parent="${namespace}/base_link"
     mass_rotor="${mass_rotor}"
@@ -169,6 +181,7 @@
     time_constant_down="${time_constant_down}"
     max_rot_velocity="${max_rot_velocity}"
-    dead_rot_velocity="${dead_rot_velocity}"
     motor_number="5"
+    rotor_drag_coefficient="${rotor_drag_coefficient}"
+    rolling_moment_coefficient="${rolling_moment_coefficient}"
     color="Red"
     use_own_mesh="false"
@@ -176,5 +189,4 @@
     <origin xyz="${cos30*arm_length} -${sin30*arm_length} ${rotor_offset_top}" rpy="0 0 0" />
     <xacro:insert_block name="rotor_inertia" />
-  </xacro:vertical_rotor_advanced>
--->
+  </xacro:vertical_rotor>
 </robot>

File: rotors_description/urdf/peregrine_base.xacro (robot description, xacro)
@@ -22,4 +22,10 @@
   <!-- Instantiate a controller. -->
   <xacro:controller_plugin_macro namespace="${namespace}" imu_sub_topic="imu" />
+  <xacro:default_camera
+    namespace="${namespace}"
+    parent_link="${namespace}/base_link"
+    camera_suffix="cam_front">
+    <origin xyz="0.35 0 0.11" rpy="0 0.2 0" />
+  </xacro:default_camera>
   <!-- Instantiate a ROS message interface -->
   <!-- <xacro:ros_interface_plugin_macro namespace="${namespace}" />-->
