Commit message: Hard coded uav_paramteres.h to use our prop-config due to parsing error. Added SITL Files (not working)

File: rotors_description/urdf/peregrineB.xacro (robot description, xacro)
@@ -41,11 +41,4 @@
   <xacro:property name="rotor_drag_coefficient" value="12.06428e-05" />
   <xacro:property name="rolling_moment_coefficient" value="0.000001" />
-  <xacro:property name="dead_rot_velocity" value="1" />
-  <!-- ############### -->
-  <!-- HIL Properties  -->
-  <!-- ############### -->
-  <xacro:property name="serial_enabled" value="true" />
-  <xacro:property name="serial_device" value="/dev/ttyACM0" />
-  <xacro:property name="enable_hil" value="true" />
   <!-- Property Blocks -->
   <xacro:property name="body_inertia">
@@ -71,77 +64,4 @@
   <!-- Instantiate rotors -->
   <gazebo>
-    <plugin name='gazebo_mavlink_interface' filename='librotors_gazebo_mavlink_interface.so'>
-      <robotNamespace>${namespace}</robotNamespace>
-      <protocol_version>2.0</protocol_version>
-      <imuSubTopic>/imu</imuSubTopic>
-      <imu_rate>250</imu_rate>
-      <gpsSubTopic>/gps</gpsSubTopic>
-      <gpsGtSubTopic>/gps_gt</gpsGtSubTopic>
-      <lidarSubTopic></lidarSubTopic>
-      <opticalFlowSubTopic></opticalFlowSubTopic>
-      <mavlink_addr>INADDR_ANY</mavlink_addr>
-      <mavlink_udp_port>14560</mavlink_udp_port>
-      <serialEnabled>true</serialEnabled>
-      <serialDevice>${serial_device}</serialDevice> <!-- Port wo pixhawk angeschlossen ist-->
-      <qgc_udp_port>14550</qgc_udp_port>
-      <hil_mode>${enable_hil}</hil_mode>
-      <baudRate>921600</baudRate>
-      <qgc_addr>INADDR_ANY</qgc_addr>
-      <hil_state_level>false</hil_state_level>
-      <enable_lockstep>false</enable_lockstep>
-      <use_tcp>false</use_tcp>
-      <motorSpeedCommandPubTopic>/gazebo/command/motor_speed_old</motorSpeedCommandPubTopic>
-      <actuatorsPubTopic>/gazebo/command/motor_speed</actuatorsPubTopic>
-      <control_channels>
-        <channel name='rotor1'>
-          <input_index>0</input_index>
-          <input_offset>0</input_offset>
-          <input_scaling>${max_rot_velocity}</input_scaling>   <!-- max rad/s  [rad/s]-->
-          <zero_position_disarmed>0</zero_position_disarmed>
-          <zero_position_armed>0</zero_position_armed>
-          <joint_control_type>gz_msg</joint_control_type>
-        </channel>
-        <channel name='rotor2'>
-          <input_index>1</input_index>
-          <input_offset>0</input_offset>
-          <input_scaling>${max_rot_velocity}</input_scaling>
-          <zero_position_disarmed>0</zero_position_disarmed>
-          <zero_position_armed>0</zero_position_armed>
-          <joint_control_type>gz_msg</joint_control_type>
-        </channel>
-        <channel name='rotor3'>
-          <input_index>2</input_index>
-          <input_offset>0</input_offset>
-          <input_scaling>${max_rot_velocity}</input_scaling>
-          <zero_position_disarmed>0</zero_position_disarmed>
-          <zero_position_armed>0</zero_position_armed>
-          <joint_control_type>gz_msg</joint_control_type>
-        </channel>
-        <channel name='rotor4'>
-          <input_index>3</input_index>
-          <input_offset>0</input_offset>
-          <input_scaling>${max_rot_velocity}</input_scaling>
-          <zero_position_disarmed>0</zero_position_disarmed>
-          <zero_position_armed>0</zero_position_armed>
-          <joint_control_type>gz_msg</joint_control_type>
-        </channel>
-        <channel name='rotor5'>
-          <input_index>5</input_index>
-          <input_offset>0</input_offset>
-          <input_scaling>${max_rot_velocity}</input_scaling>
-          <zero_position_disarmed>0</zero_position_disarmed>
-          <zero_position_armed>0</zero_position_armed>
-          <joint_control_type>gz_msg</joint_control_type>
-        </channel>
-        <channel name='rotor6'>
-          <input_index>5</input_index>
-          <input_offset>0</input_offset>
-          <input_scaling>${max_rot_velocity}</input_scaling>
-          <zero_position_disarmed>0</zero_position_disarmed>
-          <zero_position_armed>0</zero_position_armed>
-          <joint_control_type>gz_msg</joint_control_type>
-        </channel>
-      </control_channels>
-    </plugin>
     <plugin name="${namespace}_propulsion" filename="librotors_gazebo_propulsion_plugin.so">
       <robotNamespace>${namespace}</robotNamespace>
@@ -316,3 +236,4 @@
     <xacro:insert_block name="rotor_inertia" />
   </xacro:vertical_rotor_advanced>
+-->
 </robot>

File: rotors_description/urdf/peregrineB_base.xacro (robot description, xacro)
@@ -19,10 +19,18 @@
   <xacro:include filename="$(find rotors_description)/urdf/component_snippets.xacro" />
   <!-- Instantiate peregrine "mechanics" -->
-  <xacro:include filename="$(find rotors_description)/urdf/peregrine.xacro" />
-  <!-- Instantiate a controller.
+  <xacro:include filename="$(find rotors_description)/urdf/peregrineB.xacro" />
+  <!-- Instantiate a controller. -->
   <xacro:controller_plugin_macro namespace="${namespace}" imu_sub_topic="imu" />
-  -->
+  <xacro:default_camera
+    namespace="${namespace}"
+    parent_link="${namespace}/base_link"
+    camera_suffix="cam_front">
+    <origin xyz="0.35 0 0.11" rpy="0 0.2 0" />
+  </xacro:default_camera>
   <!-- Instantiate a ROS message interface -->
-  <!-- <xacro:ros_interface_plugin_macro namespace="${namespace}" />-->
+  <!-- <xacro:ros_interface_plugin_macro namespace="${namespace}" /> -->
+  <xacro:if value="$(arg enable_mavlink_interface)">
+    <xacro:default_mavlink_interface namespace="${namespace}" imu_sub_topic="imu" rotor_count="6" />
+  </xacro:if>
   <xacro:default_imu namespace="${namespace}" parent_link="${namespace}/base_link" />
   <xacro:if value="$(arg enable_ground_truth)">
