Commit message: Added the possibility to include an offset target in the peregrine.xacro

File: rotors_description/urdf/multirotor_base.xacro (robot description, xacro)
@@ -30,4 +30,31 @@
       <xacro:box_inertia x="${x}" y="${y}" z="${z}" mass="${mass}" />
     </inertial>
+  </xacro:macro>
+  <xacro:macro name="offset_target" params="namespace Ixx Iyy Izz mass parent_link *origin" >
+    <link name="${namespace}/offset_target_link">
+      <collision>
+        <origin xyz="0 0 0" rpy="0 0 0" />
+        <geometry>
+            <cylinder radius="0.2" length="0.1"/>
+        </geometry>
+      </collision>
+      <visual>
+        <origin xyz="0 0 0" rpy="0 0 0" />
+        <geometry>
+          <cylinder radius="0.1" length="0.05"/>
+        </geometry>
+        <material name="red" />
+      </visual>
+      <inertial>
+        <mass value="${mass}" />
+        <origin xyz="0 0 0" rpy="0 0 0" />
+        <inertia ixx="${Ixx}" ixy="0" ixz="0" iyy="${Iyy}" iyz="0" izz="${Izz}" />
+      </inertial>
+    </link>
+    <joint name="${namespace}/offset_target_joint" type="fixed">
+      <xacro:insert_block name="origin" />
+      <parent link="${parent_link}" />
+      <child link="${namespace}/offset_target_link" />
+    </joint>
   </xacro:macro>
   <!-- Main multirotor link -->

File: rotors_description/urdf/peregrine.xacro (robot description, xacro)
@@ -23,5 +23,5 @@
   <xacro:property name="use_mesh_file" value="true" />
   <xacro:property name="mesh_file" value="package://rotors_description/meshes/peregrine.dae" />
-  <!-- Params to be adjusted from firefly to peregrine -->
+  <!-- Params for peregrine -->
   <xacro:property name="mass" value="4.6" /> <!-- [kg] -->
   <xacro:property name="body_width" value="0.3" /> <!-- [m] -->
@@ -29,4 +29,12 @@
   <xacro:property name="mass_rotor" value="0.008" /> <!-- [kg] -->
   <xacro:property name="arm_length" value="0.42" /> <!-- [m] -->
+  <!-- Params for the target caught at an offset -->
+  <xacro:property name="offset_mass" value="0.8" /> <!-- [kg] -->
+  <xacro:property name="offset_x" value="0.3" /> <!-- [m] -->
+  <xacro:property name="offset_y" value="0.3" /> <!-- [m] -->
+  <xacro:property name="offset_z" value="0.3" /> <!-- [m] -->
+  <xacro:property name="offset_Ixx" value="0.02" /> <!-- [m] -->
+  <xacro:property name="offset_Iyy" value="0.02" /> <!-- [m] -->
+  <xacro:property name="offset_Izz" value="0.05" /> <!-- [m] -->
   <!-- this moight cause problems because negative -->
   <xacro:property name="rotor_offset_top" value="-0.05" /> <!-- [m] -->
@@ -65,4 +73,13 @@
     <xacro:insert_block name="body_inertia" />
   </xacro:multirotor_base_macro>
+  <!-- <xacro:offset_target
+    namespace="${namespace}"
+    Ixx="${offset_Ixx}"
+    Iyy="${offset_Iyy}"
+    Izz="${offset_Izz}"
+    mass="${offset_mass}"
+    parent_link="${namespace}/base_link">
+    <origin xyz="${offset_x} ${offset_y} ${offset_z}" rpy="0 0 0" />
+  </xacro:offset_target> -->
   <!-- Instantiate rotors -->
   <xacro:vertical_rotor
