Commit message: Added MPC Controller and cleaned up

File: rotors_description/urdf/peregrine.xacro (robot description, xacro)
@@ -31,21 +31,10 @@
   <xacro:property name="rotor_offset_top" value="-0.05" /> <!-- [m] -->
   <xacro:property name="radius_rotor" value="0.1778" /> <!-- [m] -->
-  <xacro:property name="motor_constant" value="4.0879e-5" /> <!-- [kg m/s^2] -->
-  <xacro:property name="moment_constant" value="0.0247" /> <!-- [m] -->
-  <xacro:property name="time_constant_up" value="0.02" /> <!-- [s] -->
-  <xacro:property name="time_constant_down" value="0.01" /> <!-- [s] -->
+  <xacro:property name="time_constant_up" value="0.05" /> <!-- [s] -->
+  <xacro:property name="time_constant_down" value="0.15" /> <!-- [s] -->
   <xacro:property name="max_rot_velocity" value="838" /> <!-- [rad/s] euals 8000rpm -->
   <xacro:property name="dead_rot_velocity" value="1" />
   <xacro:property name="sin30" value="0.5" />
   <xacro:property name="cos30" value="0.866025403784" />
-  <xacro:property name="rotor_drag_coefficient" value="12.06428e-05" />
-  <xacro:property name="rolling_moment_coefficient" value="0.000001" />
-  <xacro:property name="dead_rot_velocity" value="1" />
-  <!-- ############### -->
-  <!-- HIL Properties  -->
-  <!-- ############### -->
-  <xacro:property name="serial_enabled" value="false" />
-  <xacro:property name="serial_device" value="/dev/ttyACM0" />
-  <xacro:property name="enable_hil" value="false" />
   <!-- Property Blocks -->
   <xacro:property name="body_inertia">
@@ -71,76 +60,4 @@
   <!-- Instantiate rotors -->
   <gazebo>
-    <plugin name='gazebo_mavlink_interface' filename='librotors_gazebo_mavlink_interface.so'>
-      <robotNamespace>${namespace}</robotNamespace>
-      <protocol_version>2.0</protocol_version>
-      <imuSubTopic>/imu</imuSubTopic>
-      <imu_rate>100</imu_rate>
-      <gpsSubTopic>/gps_hil</gpsSubTopic>
-      <gpsGtSubTopic>/gps_gt</gpsGtSubTopic>
-      <lidarSubTopic></lidarSubTopic>
-      <opticalFlowSubTopic></opticalFlowSubTopic>
-      <motorSpeedCommandPubTopic>/gazebo/command/motor_speed</motorSpeedCommandPubTopic>
-      <actuatorsPubTopic>/gazebo/command/actuator_speed</actuatorsPubTopic>
-      <mavlink_addr>INADDR_ANY</mavlink_addr>
-      <mavlink_udp_port>14560</mavlink_udp_port>
-      <baudRate>921600</baudRate>
-      <qgc_addr>INADDR_ANY</qgc_addr>
-      <qgc_udp_port>14556</qgc_udp_port>
-      <hil_mode>0</hil_mode>
-      <hil_state_level>false</hil_state_level>
-      <enable_lockstep>false</enable_lockstep>
-      <use_tcp>true</use_tcp>
-      <mavlink_tcp_port>4560</mavlink_tcp_port>
-      <control_channels>
-        <channel name='rotor1'>
-          <input_index>0</input_index>
-          <input_offset>0</input_offset>
-          <input_scaling>${max_rot_velocity}</input_scaling>   <!-- max rad/s  [rad/s]-->
-          <zero_position_disarmed>0</zero_position_disarmed>
-          <zero_position_armed>0</zero_position_armed>
-          <joint_control_type>gz_msg</joint_control_type>
-        </channel>
-        <channel name='rotor2'>
-          <input_index>1</input_index>
-          <input_offset>0</input_offset>
-          <input_scaling>${max_rot_velocity}</input_scaling>
-          <zero_position_disarmed>0</zero_position_disarmed>
-          <zero_position_armed>0</zero_position_armed>
-          <joint_control_type>gz_msg</joint_control_type>
-        </channel>
-        <channel name='rotor3'>
-          <input_index>2</input_index>
-          <input_offset>0</input_offset>
-          <input_scaling>${max_rot_velocity}</input_scaling>
-          <zero_position_disarmed>0</zero_position_disarmed>
-          <zero_position_armed>0</zero_position_armed>
-          <joint_control_type>gz_msg</joint_control_type>
-        </channel>
-        <channel name='rotor4'>
-          <input_index>3</input_index>
-          <input_offset>0</input_offset>
-          <input_scaling>${max_rot_velocity}</input_scaling>
-          <zero_position_disarmed>0</zero_position_disarmed>
-          <zero_position_armed>0</zero_position_armed>
-          <joint_control_type>gz_msg</joint_control_type>
-        </channel>
-        <channel name='rotor5'>
-          <input_index>5</input_index>
-          <input_offset>0</input_offset>
-          <input_scaling>${max_rot_velocity}</input_scaling>
-          <zero_position_disarmed>0</zero_position_disarmed>
-          <zero_position_armed>0</zero_position_armed>
-          <joint_control_type>gz_msg</joint_control_type>
-        </channel>
-        <channel name='rotor6'>
-          <input_index>5</input_index>
-          <input_offset>0</input_offset>
-          <input_scaling>${max_rot_velocity}</input_scaling>
-          <zero_position_disarmed>0</zero_position_disarmed>
-          <zero_position_armed>0</zero_position_armed>
-          <joint_control_type>gz_msg</joint_control_type>
-        </channel>
-      </control_channels>
-    </plugin>
     <plugin name="${namespace}_propulsion" filename="librotors_gazebo_propulsion_plugin.so">
       <robotNamespace>${namespace}</robotNamespace>
@@ -315,3 +232,4 @@
     <xacro:insert_block name="rotor_inertia" />
   </xacro:vertical_rotor_advanced>
+-->
 </robot>

File: rotors_description/urdf/peregrine_SITL.xacro (robot description, xacro)
@@ -41,4 +41,11 @@
   <xacro:property name="rotor_drag_coefficient" value="12.06428e-05" />
   <xacro:property name="rolling_moment_coefficient" value="0.000001" />
+  <xacro:property name="dead_rot_velocity" value="1" />
+  <!-- ############### -->
+  <!-- HIL Properties  -->
+  <!-- ############### -->
+  <xacro:property name="serial_enabled" value="false" />
+  <xacro:property name="serial_device" value="/dev/ttyACM0" />
+  <xacro:property name="enable_hil" value="false" />
   <!-- Property Blocks -->
   <xacro:property name="body_inertia">
@@ -64,4 +71,76 @@
   <!-- Instantiate rotors -->
   <gazebo>
+    <plugin name='gazebo_mavlink_interface' filename='librotors_gazebo_mavlink_interface.so'>
+      <robotNamespace>${namespace}</robotNamespace>
+      <protocol_version>2.0</protocol_version>
+      <imuSubTopic>/imu</imuSubTopic>
+      <imu_rate>100</imu_rate>
+      <gpsSubTopic>/gps_hil</gpsSubTopic>
+      <gpsGtSubTopic>/gps_gt</gpsGtSubTopic>
+      <lidarSubTopic></lidarSubTopic>
+      <opticalFlowSubTopic></opticalFlowSubTopic>
+      <motorSpeedCommandPubTopic>/gazebo/command/motor_speed</motorSpeedCommandPubTopic>
+      <actuatorsPubTopic>/gazebo/command/actuator_speed</actuatorsPubTopic>
+      <mavlink_addr>INADDR_ANY</mavlink_addr>
+      <mavlink_udp_port>14560</mavlink_udp_port>
+      <baudRate>921600</baudRate>
+      <qgc_addr>INADDR_ANY</qgc_addr>
+      <qgc_udp_port>14556</qgc_udp_port>
+      <hil_mode>0</hil_mode>
+      <hil_state_level>false</hil_state_level>
+      <enable_lockstep>false</enable_lockstep>
+      <use_tcp>true</use_tcp>
+      <mavlink_tcp_port>4560</mavlink_tcp_port>
+      <control_channels>
+        <channel name='rotor1'>
+          <input_index>0</input_index>
+          <input_offset>0</input_offset>
+          <input_scaling>${max_rot_velocity}</input_scaling>   <!-- max rad/s  [rad/s]-->
+          <zero_position_disarmed>0</zero_position_disarmed>
+          <zero_position_armed>0</zero_position_armed>
+          <joint_control_type>gz_msg</joint_control_type>
+        </channel>
+        <channel name='rotor2'>
+          <input_index>1</input_index>
+          <input_offset>0</input_offset>
+          <input_scaling>${max_rot_velocity}</input_scaling>
+          <zero_position_disarmed>0</zero_position_disarmed>
+          <zero_position_armed>0</zero_position_armed>
+          <joint_control_type>gz_msg</joint_control_type>
+        </channel>
+        <channel name='rotor3'>
+          <input_index>2</input_index>
+          <input_offset>0</input_offset>
+          <input_scaling>${max_rot_velocity}</input_scaling>
+          <zero_position_disarmed>0</zero_position_disarmed>
+          <zero_position_armed>0</zero_position_armed>
+          <joint_control_type>gz_msg</joint_control_type>
+        </channel>
+        <channel name='rotor4'>
+          <input_index>3</input_index>
+          <input_offset>0</input_offset>
+          <input_scaling>${max_rot_velocity}</input_scaling>
+          <zero_position_disarmed>0</zero_position_disarmed>
+          <zero_position_armed>0</zero_position_armed>
+          <joint_control_type>gz_msg</joint_control_type>
+        </channel>
+        <channel name='rotor5'>
+          <input_index>5</input_index>
+          <input_offset>0</input_offset>
+          <input_scaling>${max_rot_velocity}</input_scaling>
+          <zero_position_disarmed>0</zero_position_disarmed>
+          <zero_position_armed>0</zero_position_armed>
+          <joint_control_type>gz_msg</joint_control_type>
+        </channel>
+        <channel name='rotor6'>
+          <input_index>5</input_index>
+          <input_offset>0</input_offset>
+          <input_scaling>${max_rot_velocity}</input_scaling>
+          <zero_position_disarmed>0</zero_position_disarmed>
+          <zero_position_armed>0</zero_position_armed>
+          <joint_control_type>gz_msg</joint_control_type>
+        </channel>
+      </control_channels>
+    </plugin>
     <plugin name="${namespace}_propulsion" filename="librotors_gazebo_propulsion_plugin.so">
       <robotNamespace>${namespace}</robotNamespace>
@@ -236,4 +315,3 @@
     <xacro:insert_block name="rotor_inertia" />
   </xacro:vertical_rotor_advanced>
--->
 </robot>

File: rotors_description/urdf/peregrine_base.xacro (robot description, xacro)
@@ -20,9 +20,11 @@
   <!-- Instantiate peregrine "mechanics" -->
   <xacro:include filename="$(find rotors_description)/urdf/peregrine.xacro" />
-  <!-- Instantiate a controller.
+  <!-- Instantiate a controller. -->
   <xacro:controller_plugin_macro namespace="${namespace}" imu_sub_topic="imu" />
-  -->
   <!-- Instantiate a ROS message interface -->
-  <!-- <xacro:ros_interface_plugin_macro namespace="${namespace}" />-->
+  <!-- <xacro:ros_interface_plugin_macro namespace="${namespace}" /> -->
+  <xacro:if value="$(arg enable_mavlink_interface)">
+    <xacro:default_mavlink_interface namespace="${namespace}" imu_sub_topic="imu" rotor_count="6" />
+  </xacro:if>
   <xacro:default_imu namespace="${namespace}" parent_link="${namespace}/base_link" />
   <xacro:default_gps namespace="${namespace}" parent_link="${namespace}/base_link" />

File: rotors_description/urdf/peregrine_base_SITL.xacro (robot description, xacro)
@@ -19,19 +19,12 @@
   <xacro:include filename="$(find rotors_description)/urdf/component_snippets.xacro" />
   <!-- Instantiate peregrine "mechanics" -->
-  <xacro:include filename="$(find rotors_description)/urdf/peregrineB.xacro" />
-  <!-- Instantiate a controller. -->
+  <xacro:include filename="$(find rotors_description)/urdf/peregrine.xacro" />
+  <!-- Instantiate a controller.
   <xacro:controller_plugin_macro namespace="${namespace}" imu_sub_topic="imu" />
-  <xacro:default_camera
-    namespace="${namespace}"
-    parent_link="${namespace}/base_link"
-    camera_suffix="cam_front">
-    <origin xyz="0.35 0 0.11" rpy="0 0.2 0" />
-  </xacro:default_camera>
+  -->
   <!-- Instantiate a ROS message interface -->
-  <!-- <xacro:ros_interface_plugin_macro namespace="${namespace}" /> -->
-  <xacro:if value="$(arg enable_mavlink_interface)">
-    <xacro:default_mavlink_interface namespace="${namespace}" imu_sub_topic="imu" rotor_count="6" />
-  </xacro:if>
+  <!-- <xacro:ros_interface_plugin_macro namespace="${namespace}" />-->
   <xacro:default_imu namespace="${namespace}" parent_link="${namespace}/base_link" />
+  <xacro:default_gps namespace="${namespace}" parent_link="${namespace}/base_link" />
   <xacro:if value="$(arg enable_ground_truth)">
     <xacro:ground_truth_imu_and_odometry namespace="${namespace}" parent_link="${namespace}/base_link" />

File: rotors_description/urdf/peregrine_base_or.xacro (robot description, xacro)
@@ -19,5 +19,5 @@
   <xacro:include filename="$(find rotors_description)/urdf/component_snippets.xacro" />
   <!-- Instantiate peregrine "mechanics" -->
-  <xacro:include filename="$(find rotors_description)/urdf/peregrineA.xacro" />
+  <xacro:include filename="$(find rotors_description)/urdf/peregrine.xacro" />
   <!-- Instantiate a controller. -->
   <xacro:controller_plugin_macro namespace="${namespace}" imu_sub_topic="imu" />
@@ -29,4 +29,5 @@
   </xacro:if>
   <xacro:default_imu namespace="${namespace}" parent_link="${namespace}/base_link" />
+  <xacro:default_gps namespace="${namespace}" parent_link="${namespace}/base_link" />
   <xacro:if value="$(arg enable_ground_truth)">
     <xacro:ground_truth_imu_and_odometry namespace="${namespace}" parent_link="${namespace}/base_link" />

Commit message: compared params in xacro and control files

File: rotors_description/urdf/peregrine.xacro (robot description, xacro)
@@ -28,5 +28,5 @@
   <xacro:property name="body_height" value="0.3" /> <!-- [m] -->
   <xacro:property name="mass_rotor" value="0.008" /> <!-- [kg] -->
-  <xacro:property name="arm_length" value="0.4" /> <!-- [m] -->
+  <xacro:property name="arm_length" value="0.42" /> <!-- [m] -->
   <!-- this moight cause problems because negative -->
   <xacro:property name="rotor_offset_top" value="-0.05" /> <!-- [m] -->

Commit message: change in peregrinne. xacro

File: rotors_description/urdf/peregrine.xacro (robot description, xacro)
@@ -24,5 +24,5 @@
   <xacro:property name="mesh_file" value="package://rotors_description/meshes/peregrine.dae" />
   <!-- Params for peregrine -->
-  <xacro:property name="mass" value="4.6" /> <!-- [kg] -->
+  <xacro:property name="mass" value="6.0" /> <!-- [kg] -->
   <xacro:property name="body_width" value="0.3" /> <!-- [m] -->
   <xacro:property name="body_height" value="0.3" /> <!-- [m] -->
@@ -30,5 +30,5 @@
   <xacro:property name="arm_length" value="0.42" /> <!-- [m] -->
   <!-- Params for the target caught at an offset -->
-  <xacro:property name="offset_mass" value="0.8" /> <!-- [kg] -->
+  <xacro:property name="offset_mass" value="0.0" /> <!-- [kg] -->
   <xacro:property name="offset_x" value="0.3" /> <!-- [m] -->
   <xacro:property name="offset_y" value="0.3" /> <!-- [m] -->

Commit message: redo changes from previous commit

File: rotors_description/urdf/peregrine.xacro (robot description, xacro)
@@ -24,5 +24,5 @@
   <xacro:property name="mesh_file" value="package://rotors_description/meshes/peregrine.dae" />
   <!-- Params for peregrine -->
-  <xacro:property name="mass" value="6.0" /> <!-- [kg] -->
+  <xacro:property name="mass" value="4.6" /> <!-- [kg] -->
   <xacro:property name="body_width" value="0.3" /> <!-- [m] -->
   <xacro:property name="body_height" value="0.3" /> <!-- [m] -->
@@ -30,5 +30,5 @@
   <xacro:property name="arm_length" value="0.42" /> <!-- [m] -->
   <!-- Params for the target caught at an offset -->
-  <xacro:property name="offset_mass" value="0.0" /> <!-- [kg] -->
+  <xacro:property name="offset_mass" value="0.00" /> <!-- [kg] -->
   <xacro:property name="offset_x" value="0.3" /> <!-- [m] -->
   <xacro:property name="offset_y" value="0.3" /> <!-- [m] -->

Commit message: Subscriber doesn't work

File: rotors_description/urdf/peregrine.xacro (robot description, xacro)
@@ -29,12 +29,4 @@
   <xacro:property name="mass_rotor" value="0.008" /> <!-- [kg] -->
   <xacro:property name="arm_length" value="0.42" /> <!-- [m] -->
-  <!-- Params for the target caught at an offset -->
-  <xacro:property name="offset_mass" value="0.00" /> <!-- [kg] -->
-  <xacro:property name="offset_x" value="0.3" /> <!-- [m] -->
-  <xacro:property name="offset_y" value="0.3" /> <!-- [m] -->
-  <xacro:property name="offset_z" value="0.3" /> <!-- [m] -->
-  <xacro:property name="offset_Ixx" value="0.02" /> <!-- [m] -->
-  <xacro:property name="offset_Iyy" value="0.02" /> <!-- [m] -->
-  <xacro:property name="offset_Izz" value="0.05" /> <!-- [m] -->
   <!-- this moight cause problems because negative -->
   <xacro:property name="rotor_offset_top" value="-0.05" /> <!-- [m] -->
@@ -73,13 +65,4 @@
     <xacro:insert_block name="body_inertia" />
   </xacro:multirotor_base_macro>
-  <!-- <xacro:offset_target
-    namespace="${namespace}"
-    Ixx="${offset_Ixx}"
-    Iyy="${offset_Iyy}"
-    Izz="${offset_Izz}"
-    mass="${offset_mass}"
-    parent_link="${namespace}/base_link">
-    <origin xyz="${offset_x} ${offset_y} ${offset_z}" rpy="0 0 0" />
-  </xacro:offset_target> -->
   <!-- Instantiate rotors -->
   <xacro:vertical_rotor
@@ -207,3 +190,51 @@
     <xacro:insert_block name="rotor_inertia" />
   </xacro:vertical_rotor>
+  <!-- Payload -->
+  <link name="${namespace}/target_drone">
+     <inertial>
+        <origin xyz="0.01 0 0" rpy="0 0 0" />
+        <mass value="1" />
+        <inertia ixx="0.02" ixy="0.0" ixz="0.0" iyy="0.02" iyz="0.0" izz="0.05" /> <!-- [kg m^2] [kg m^2] [kg m^2] [kg m^2] [kg m^2] [kg m^2] -->
+     </inertial>
+     <visual>
+        <origin xyz="0.01 0 0" rpy="0 0 0" />
+        <geometry>
+           <!-- <mesh filename="package://rotors_description/meshes/payloads/payload.stl" scale="0.012 0.012 0.012" /> -->
+           <cylinder length="0.1" radius="0.25"/>
+        </geometry>
+     </visual>
+     <collision>
+        <origin xyz="0.01 0 0" rpy="0 0 0" />
+        <geometry>
+          <cylinder length="0.1" radius="0.25"/>
+        </geometry>
+     </collision>
+  </link>
+  <joint name="${namespace}/target_drone_joint" type="floating">
+     <parent link="${namespace}/base_link" />
+     <child link="${namespace}/target_drone" />
+     <origin xyz="0 0 0" rpy="0 0 0" />
+  </joint>
+  <gazebo reference="${namespace}/target_drone">
+     <visual>
+        <!-- <plugin name="visual_plugin_target_drone" filename="librotors_gazebo_template_visual_plugin.so" /> -->
+        <cylinder length="0.1" radius="0.25"/>
+     </visual>
+     <material>Gazebo/Orange</material>
+     <mu1>0.2</mu1>
+     <mu2>0.2</mu2>
+     <kp>10000</kp>
+     <kd>1</kd>
+  </gazebo>
+  <gazebo>
+     <plugin filename="librotors_gazebo_payload_plugin.so" name="payload_plugin">
+        <robotNamespace>${namespace}</robotNamespace>
+        <joint>${namespace}/payload_1_joint</joint>
+        <payload>${namespace}/target_drone</payload>
+        <parent>${namespace}/base_link</parent>
+        <hoistPosParent>0 -0.15 -0.04</hoistPosParent>
+        <hoistPosPayload>0 0 0</hoistPosPayload>
+        <dropTopic>drop_1</dropTopic>
+     </plugin>
+  </gazebo>
 </robot>
