Commit message: Clean Up Believer Aerodynamic Model, Discard Dihedral, Add yaml files for believer

File: rotors_description/urdf/believer.xacro (robot description, xacro)
@@ -365,7 +365,7 @@
           <forward>1 0 0</forward>
           <upward>0 0 1</upward>
-          <cp>0.075 0.075 0.0</cp>
-          <seg_area>0.06</seg_area>
-          <seg_chord>0.236</seg_chord>
+          <cp>0.0 0.143 0.025</cp>
+          <seg_area>0.042</seg_area>
+          <seg_chord>0.292</seg_chord>
           <aeroParamsYAML>${yaml_path}/believer_wing.yaml</aeroParamsYAML>
           <wind name="wind">
@@ -376,11 +376,14 @@
           <forward>1 0 0</forward>
           <upward>0 0 1</upward>
-          <cp>0.06 0.24 0.0</cp>
-          <seg_area>0.06</seg_area>
-          <seg_chord>0.183</seg_chord>
-          <aeroParamsYAML>${yaml_path}/believer_wing.yaml</aeroParamsYAML>
-          <wind name="wind">
-            <topic>wind_base_link</topic>
-          </wind>
+          <cp>0.0 0.287 0.025</cp>
+          <seg_area>0.041</seg_area>
+          <seg_chord>0.287</seg_chord>
+          <aeroParamsYAML>${yaml_path}/believer_wing.yaml</aeroParamsYAML>
+          <wind name="wind">
+            <topic>wind_base_link</topic>
+          </wind>
+          <indVel name="prop0">
+            <topic>prop_slpstr_0</topic>
+          </indVel>
           <control>
             <cs name="flap_left">
@@ -393,11 +396,14 @@
           <forward>1 0 0</forward>
           <upward>0 0 1</upward>
-          <cp>0.05 0.36 0.0</cp>
-          <seg_area>0.06</seg_area>
-          <seg_chord>0.236</seg_chord>
-          <aeroParamsYAML>${yaml_path}/believer_wing.yaml</aeroParamsYAML>
-          <wind name="wind">
-            <topic>wind_base_link</topic>
-          </wind>
+          <cp>0.0 0.43 0.025</cp>
+          <seg_area>0.04</seg_area>
+          <seg_chord>0.28</seg_chord>
+          <aeroParamsYAML>${yaml_path}/believer_wing.yaml</aeroParamsYAML>
+          <wind name="wind">
+            <topic>wind_base_link</topic>
+          </wind>
+          <indVel name="prop0">
+            <topic>prop_slpstr_0</topic>
+          </indVel>
           <control>
             <cs name="flap_left">
@@ -410,7 +416,7 @@
           <forward>1 0 0</forward>
           <upward>0 0 1</upward>
-          <cp>0.04 0.52 0.02</cp>
-          <seg_area>0.06</seg_area>
-          <seg_chord>0.236</seg_chord>
+          <cp>0.0 0.57 0.025</cp>
+          <seg_area>0.036</seg_area>
+          <seg_chord>0.253</seg_chord>
           <aeroParamsYAML>${yaml_path}/believer_wing.yaml</aeroParamsYAML>
           <wind name="wind">
@@ -421,7 +427,7 @@
           <forward>1 0 0</forward>
           <upward>0 0 1</upward>
-          <cp>0.03 0.6 0.06</cp>
-          <seg_area>0.043</seg_area>
-          <seg_chord>0.236</seg_chord>
+          <cp>0.0 0.72 0.03</cp>
+          <seg_area>0.035</seg_area>
+          <seg_chord>0.245</seg_chord>
           <aeroParamsYAML>${yaml_path}/believer_wing.yaml</aeroParamsYAML>
           <wind name="wind">
@@ -438,7 +444,7 @@
           <forward>1 0 0</forward>
           <upward>0 0 1</upward>
-          <cp>0.03 0.78 0.1</cp>
-          <seg_area>0.043</seg_area>
-          <seg_chord>0.236</seg_chord>
+          <cp>-0.03 0.84 0.04</cp>
+          <seg_area>0.033</seg_area>
+          <seg_chord>0.234</seg_chord>
           <aeroParamsYAML>${yaml_path}/believer_wing.yaml</aeroParamsYAML>
           <wind name="wind">
@@ -455,7 +461,7 @@
           <forward>1 0 0</forward>
           <upward>0 0 1</upward>
-          <cp>0.075 -0.075 0.0</cp>
-          <seg_area>0.06</seg_area>
-          <seg_chord>0.236</seg_chord>
+          <cp>0.0 -0.143 0.025</cp>
+          <seg_area>0.042</seg_area>
+          <seg_chord>0.292</seg_chord>
           <aeroParamsYAML>${yaml_path}/believer_wing.yaml</aeroParamsYAML>
           <wind name="wind">
@@ -466,11 +472,14 @@
           <forward>1 0 0</forward>
           <upward>0 0 1</upward>
-          <cp>0.06 -0.24 0.0</cp>
-          <seg_area>0.06</seg_area>
-          <seg_chord>0.236</seg_chord>
-          <aeroParamsYAML>${yaml_path}/believer_wing.yaml</aeroParamsYAML>
-          <wind name="wind">
-            <topic>wind_base_link</topic>
-          </wind>
+          <cp>0.0 -0.287 0.025</cp>
+          <seg_area>0.041</seg_area>
+          <seg_chord>0.287</seg_chord>
+          <aeroParamsYAML>${yaml_path}/believer_wing.yaml</aeroParamsYAML>
+          <wind name="wind">
+            <topic>wind_base_link</topic>
+          </wind>
+          <indVel name="prop1">
+            <topic>prop_slpstr_1</topic>
+          </indVel>
           <control>
             <cs name="flap_right">
@@ -483,11 +492,14 @@
           <forward>1 0 0</forward>
           <upward>0 0 1</upward>
-          <cp>0.05 -0.36 0.0</cp>
-          <seg_area>0.06</seg_area>
-          <seg_chord>0.236</seg_chord>
-          <aeroParamsYAML>${yaml_path}/believer_wing.yaml</aeroParamsYAML>
-          <wind name="wind">
-            <topic>wind_base_link</topic>
-          </wind>
+          <cp>0.0 -0.43 0.025</cp>
+          <seg_area>0.04</seg_area>
+          <seg_chord>0.28</seg_chord>
+          <aeroParamsYAML>${yaml_path}/believer_wing.yaml</aeroParamsYAML>
+          <wind name="wind">
+            <topic>wind_base_link</topic>
+          </wind>
+          <indVel name="prop1">
+            <topic>prop_slpstr_1</topic>
+          </indVel>
           <control>
             <cs name="flap_right">
@@ -500,7 +512,7 @@
           <forward>1 0 0</forward>
           <upward>0 0 1</upward>
-          <cp>0.04 -0.52 0.02</cp>
-          <seg_area>0.06</seg_area>
-          <seg_chord>0.236</seg_chord>
+          <cp>0.0 -0.57 0.025</cp>
+          <seg_area>0.036</seg_area>
+          <seg_chord>0.253</seg_chord>
           <aeroParamsYAML>${yaml_path}/believer_wing.yaml</aeroParamsYAML>
           <wind name="wind">
@@ -511,7 +523,7 @@
           <forward>1 0 0</forward>
           <upward>0 0 1</upward>
-          <cp>0.03 -0.6 0.06</cp>
-          <seg_area>0.043</seg_area>
-          <seg_chord>0.236</seg_chord>
+          <cp>0.0 -0.72 0.03</cp>
+          <seg_area>0.035</seg_area>
+          <seg_chord>0.245</seg_chord>
           <aeroParamsYAML>${yaml_path}/believer_wing.yaml</aeroParamsYAML>
           <wind name="wind">
@@ -528,7 +540,7 @@
           <forward>1 0 0</forward>
           <upward>0 0 1</upward>
-          <cp>0.03 -0.78 0.1</cp>
-          <seg_area>0.043</seg_area>
-          <seg_chord>0.236</seg_chord>
+          <cp>-0.03 -0.84 0.04</cp>
+          <seg_area>0.033</seg_area>
+          <seg_chord>0.234</seg_chord>
           <aeroParamsYAML>${yaml_path}/believer_wing.yaml</aeroParamsYAML>
           <wind name="wind">
@@ -603,5 +615,5 @@
       <qgc_udp_port>14550</qgc_udp_port>
       <hil_mode>true</hil_mode>
-      <hil_state_level>true</hil_state_level>
+      <hil_state_level>false</hil_state_level>
       <enable_lockstep>false</enable_lockstep>
       <use_tcp>false</use_tcp>
@@ -618,5 +630,5 @@
         <input_index>4</input_index>
         <input_offset>0</input_offset>
-        <input_scaling>1185</input_scaling><!-- rdps_slope/2  [rad/s]-->
+        <input_scaling>985</input_scaling><!-- rdps_slope/2  [rad/s]-->
         <zero_position_disarmed>0</zero_position_disarmed>
         <zero_position_armed>15</zero_position_armed>
@@ -636,5 +648,5 @@
         <input_index>5</input_index>
         <input_offset>0</input_offset>
-        <input_scaling>1185</input_scaling><!-- rdps_slope/2  [rad/s]-->
+        <input_scaling>985</input_scaling><!-- rdps_slope/2  [rad/s]-->
         <zero_position_disarmed>0</zero_position_disarmed>
         <zero_position_armed>15</zero_position_armed>

File: rotors_description/urdf/believer_base.xacro (robot description, xacro)
@@ -28,5 +28,5 @@
     parent_link="${namespace}/base_link"
     camera_suffix="cam_front">
-    <origin xyz="0.0 0.0 -0.1" rpy="0 0.2 0" />
+    <origin xyz="0.465 0 0.05" rpy="0 0.2 0" />
   </xacro:default_camera>
 </robot>

Commit message: Add payload and lidar

File: rotors_description/urdf/believer.xacro (robot description, xacro)
@@ -103,4 +103,5 @@
   <!-- Included URDF Files -->
   <xacro:include filename="$(find rotors_description)/urdf/fixed_wing_X_base.xacro" />
+  <xacro:include filename="$(find rotors_description)/urdf/hook_simple.xacro" />
   <!-- Instantiate fixed_wing_base_macro once -->
   <xacro:fixed_wing_base_macro
@@ -116,4 +117,54 @@
     <xacro:insert_block name="body_inertia" />
   </xacro:fixed_wing_base_macro>
+  <!-- <xacro:payload_hook_simple namespace="${namespace}">
+  </xacro:payload_hook_simple>
+  <link name="${namespace}/soccer_ball_1">
+    <inertial>
+       <origin xyz="0 0 0" rpy="0 0 0" />
+       <mass value="1.0" />
+       <xacro:sphere_inertia r="0.25" mass="1.0" />
+    </inertial>
+    <visual>
+       <origin xyz="0 0 0" rpy="0 0 0" />
+       <geometry>
+          <sphere radius = "0.25" />
+       </geometry>
+    </visual>
+    <collision>
+       <origin xyz="0 0 0" rpy="0 0 0" />
+       <geometry>
+          <sphere radius = "0.25" />
+       </geometry>
+    </collision>
+  </link>
+  <joint name="${namespace}/payload_1_joint" type="floating">
+    <parent link="${namespace}/payload_hook" />
+    <child link="${namespace}/soccer_ball_1" />
+    <origin xyz="-1.5 0 0" rpy="0 0 0" />
+  </joint>
+  <gazebo reference="${namespace}/soccer_ball_1">
+    <material>Gazebo/White</material>
+    <mu1>0.2</mu1>
+    <mu2>0.2</mu2>
+    <kp>10000</kp>
+    <kd>1</kd>
+  </gazebo>
+  <gazebo>
+    <plugin filename="librotors_gazebo_payload_plugin.so" name="payload_plugin_1">
+       <robotNamespace>${namespace}</robotNamespace>
+       <joint>${namespace}/payload_1_joint</joint>
+       <payload>${namespace}/soccer_ball_1</payload>
+       <parent>${namespace}/payload_hook</parent>
+       <proxRec>true</proxRec>
+       <radiusRec>0.5</radiusRec>
+       <omega>6</omega>
+       <hoistPosParent>-1.0 0 0</hoistPosParent>
+       <hoistPosPayload>0 0 0</hoistPosPayload>
+       <pickupWorldPosPayload>0 0 2.2</pickupWorldPosPayload>
+       <initialState>3</initialState>
+       <dropTopic>drop_1</dropTopic>
+       <payloadTrackingTopic>soccer_ball_1</payloadTrackingTopic>
+    </plugin>
+  </gazebo> -->
   <!-- Instantiate the ailerons -->
   <xacro:control_surface
@@ -274,14 +325,14 @@
         <windLayer>
           <layer name="layer1">
-            <altitude>10</altitude>
-            <windMeanNED>-5 0 0</windMeanNED>
+            <altitude>2</altitude>
+            <windMeanNED>-2 0 0</windMeanNED>
           </layer>
           <layer name="layer2">
-            <altitude>25</altitude>
-            <windMeanNED>-6 0 0</windMeanNED>
+            <altitude>10</altitude>
+            <windMeanNED>-4 0.5 1</windMeanNED>
           </layer>
           <layer name="layer3">
             <altitude>35</altitude>
-            <windMeanNED>-10 0 0</windMeanNED>
+            <windMeanNED>-4 0 0</windMeanNED>
           </layer>
         </windLayer>
@@ -293,8 +344,8 @@
         </findWind>
         <lambdaMin>10</lambdaMin>
-        <lengthScale>725</lengthScale>
-        <fourierNNN>10 10 10</fourierNNN>
-        <sigma>5</sigma>
-        <trnspVelTurbNED>5 0 0</trnspVelTurbNED>
+        <lengthScale>750</lengthScale>
+        <fourierNNN>5 5 5</fourierNNN>
+        <sigma>2</sigma>
+        <trnspVelTurbNED>3 0 0</trnspVelTurbNED>
       </plugin>
     </gazebo>
@@ -558,10 +609,11 @@
           <upward>0 -0.5 0.866</upward>
           <cp>-0.713 0.158 0.1</cp>
+          <!-- <cp>-0.813 0.158 0.1</cp> -->
           <seg_area>0.068</seg_area>
           <seg_chord>0.22</seg_chord>
           <aeroParamsYAML>${yaml_path}/believer_vtail.yaml</aeroParamsYAML>
-          <indVel name="prop0">
+          <!-- <indVel name="prop0">
             <topic>prop_slpstr_0</topic>
-          </indVel>
+          </indVel> -->
           <wind name="wind">
             <topic>wind_base_link</topic>
@@ -578,10 +630,11 @@
           <upward>0 0.5 0.866</upward>
           <cp>-0.713 -0.158 0.1</cp>
+          <!-- <cp>-0.813 0.158 0.1</cp> -->
           <seg_area>0.068</seg_area>
           <seg_chord>0.22</seg_chord>
           <aeroParamsYAML>${yaml_path}/believer_vtail.yaml</aeroParamsYAML>
-          <indVel name="prop1">
+          <!-- <indVel name="prop1">
             <topic>prop_slpstr_1</topic>
-          </indVel>
+          </indVel> -->
           <wind name="wind">
             <topic>wind_base_link</topic>
@@ -602,8 +655,8 @@
       <protocol_version>2.0</protocol_version>
       <imuSubTopic>/imu</imuSubTopic>
+      <lidarSubTopic>/lidar_lite_v3</lidarSubTopic>
       <imu_rate>250</imu_rate>
       <gpsSubTopic>/gps</gpsSubTopic>
       <gpsGtSubTopic>/gps_gt</gpsGtSubTopic>
-      <lidarSubTopic></lidarSubTopic>
       <opticalFlowSubTopic></opticalFlowSubTopic>
       <mavlink_addr>INADDR_ANY</mavlink_addr>

File: rotors_description/urdf/believer_base.xacro (robot description, xacro)
@@ -24,4 +24,7 @@
     <origin xyz="0.0 0.0 0.1" rpy="0 0 0" />
   </xacro:default_gps>
+  <xacro:default_lidar namespace="${namespace}" parent_link="${namespace}/base_link" >
+    <origin xyz="-0.2 0.0 -0.1" rpy="0 1.506 0" />
+  </xacro:default_lidar>
   <xacro:default_camera
     namespace="${namespace}"
